Commit message: float zero

File: melfa_description/ros2_control/rv2fr.hardware.xacro (robot description, xacro)
@@ -62,5 +62,5 @@
                 <param name="initial_position">${initial_positions['rv_joint_3']}</param>
                 <command_interface name="position" >
-                    <param name="min">0</param>
+                    <param name="min">0.0</param>
                     <param name="max">2.792526803190927</param>
                 </command_interface>

File: melfa_description/ros2_control/rv4fr.hardware.xacro (robot description, xacro)
@@ -62,5 +62,5 @@
                 <param name="initial_position">${initial_positions['rv_joint_3']}</param>
                 <command_interface name="position" >
-                    <param name="min">0</param>
+                    <param name="min">0.0</param>
                     <param name="max">2.8623399732707</param>
                 </command_interface>

File: melfa_description/ros2_control/rv4frl.hardware.xacro (robot description, xacro)
@@ -62,5 +62,5 @@
                 <param name="initial_position">${initial_positions['rv_joint_3']}</param>
                 <command_interface name="position" >
-                    <param name="min">0</param>
+                    <param name="min">0.0</param>
                     <param name="max">2.8623399732707</param>
                 </command_interface>

File: melfa_description/ros2_control/rv7frl.hardware.xacro (robot description, xacro)
@@ -62,5 +62,5 @@
                 <param name="initial_position">${initial_positions['rv_joint_3']}</param>
                 <command_interface name="position" >
-                    <param name="min">0</param>
+                    <param name="min">0.0</param>
                     <param name="max">2.827433</param>
                 </command_interface>

File: melfa_description/ros2_control/rv80fr.hardware.xacro (robot description, xacro)
@@ -62,5 +62,5 @@
                 <param name="initial_position">${initial_positions['rv_joint_3']}</param>
                 <command_interface name="position" >
-                    <param name="min">--2.356194</param>
+                    <param name="min">-2.356194</param>
                     <param name="max">2.70526</param>
                 </command_interface>

File: melfa_description/urdf/rv2fr/rv2fr_macro.xacro (robot description, xacro)
@@ -49,5 +49,5 @@
             <child link="${prefix}rv2fr_elbow"/>
             <axis xyz="0 1 0"/>
-            <limit lower="0.0" upper="2.792526803190927" effort="500" velocity="5.235987755982989"/>
+            <limit lower="0.0" upper="2.792526803190927" effort="50" velocity="5.235987755982989"/>
             <dynamics damping="1.0" friction="1.0"/>
         </joint>
