Commit message: Fix some typo.

File: melfa_description/urdf/rh6crh6020/rh6crh6020_macro.xacro (robot description, xacro)
@@ -12,5 +12,5 @@
     <xacro:macro name="rh6crh6020" params="parent prefix *origin">
             <!-- Inertial parameters -->
-        <xacro:property name="base_mass" value="0.4" />  <!-- These mass are INCORRRECT -->
+        <xacro:property name="base_mass" value="0.4" />  <!-- These mass are INCORRECT -->
         <xacro:property name="shoulder_mass" value="0.37000" />
         <xacro:property name="upper_arm_mass" value="0.83930" />

File: melfa_description/urdf/rh6frh5520/rh6frh5520_macro.xacro (robot description, xacro)
@@ -12,5 +12,5 @@
     <xacro:macro name="rh6frh5520" params="parent prefix *origin">
         <!-- Inertial parameters -->
-        <xacro:property name="base_mass" value="0.4" />  <!-- These mass are INCORRRECT -->
+        <xacro:property name="base_mass" value="0.4" />  <!-- These mass are INCORRECT -->
         <xacro:property name="shoulder_mass" value="0.37000" />
         <xacro:property name="upper_arm_mass" value="0.83930" />

File: melfa_description/urdf/rv13frl/rv13frl_macro.xacro (robot description, xacro)
@@ -12,5 +12,5 @@
     <xacro:macro name="rv13frl" params="parent prefix *origin">
         <!-- Inertial parameters -->
-        <xacro:property name="base_mass" value="0.4" />  <!-- These mass are INCORRRECT -->
+        <xacro:property name="base_mass" value="0.4" />  <!-- These mass are INCORRECT -->
         <xacro:property name="shoulder_mass" value="0.37000" />
         <xacro:property name="upper_arm_mass" value="0.33930" />

File: melfa_description/urdf/rv2fr/rv2fr_macro.xacro (robot description, xacro)
@@ -12,5 +12,5 @@
     <xacro:macro name="rv2fr" params="parent prefix *origin">
         <!-- Inertial parameters -->
-        <xacro:property name="base_mass" value="0.4" />  <!-- These mass are INCORRRECT -->
+        <xacro:property name="base_mass" value="0.4" />  <!-- These mass are INCORRECT -->
         <xacro:property name="shoulder_mass" value="0.37000" />
         <xacro:property name="upper_arm_mass" value="0.33930" />

File: melfa_description/urdf/rv4fr/rv4fr_macro.xacro (robot description, xacro)
@@ -12,5 +12,5 @@
     <xacro:macro name="rv4fr" params="parent prefix *origin">
         <!-- Inertial parameters -->
-        <xacro:property name="base_mass" value="0.4" />  <!-- These mass are INCORRRECT -->
+        <xacro:property name="base_mass" value="0.4" />  <!-- These mass are INCORRECT -->
         <xacro:property name="shoulder_mass" value="0.37000" />
         <xacro:property name="upper_arm_mass" value="0.33930" />

File: melfa_description/urdf/rv4frl/rv4frl_macro.xacro (robot description, xacro)
@@ -12,5 +12,5 @@
     <xacro:macro name="rv4frl" params="parent prefix *origin">
         <!-- Inertial parameters -->
-        <xacro:property name="base_mass" value="0.4" />  <!-- These mass are INCORRRECT -->
+        <xacro:property name="base_mass" value="0.4" />  <!-- These mass are INCORRECT -->
         <xacro:property name="shoulder_mass" value="0.37000" />
         <xacro:property name="upper_arm_mass" value="0.33930" />

File: melfa_description/urdf/rv5as/rv5as_macro.xacro (robot description, xacro)
@@ -12,5 +12,5 @@
     <xacro:macro name="rv5as" params="parent prefix *origin">
         <!-- Inertial parameters -->
-        <xacro:property name="base_mass" value="0.4" />  <!-- These mass are INCORRRECT -->
+        <xacro:property name="base_mass" value="0.4" />  <!-- These mass are INCORRECT -->
         <xacro:property name="shoulder_mass" value="0.37000" />
         <xacro:property name="upper_arm_mass" value="0.33930" />

File: melfa_description/urdf/rv7frl/rv7frl_macro.xacro (robot description, xacro)
@@ -12,5 +12,5 @@
     <xacro:macro name="rv7frl" params="parent prefix *origin">
         <!-- Inertial parameters -->
-        <xacro:property name="base_mass" value="0.4" />  <!-- These mass are INCORRRECT -->
+        <xacro:property name="base_mass" value="0.4" />  <!-- These mass are INCORRECT -->
         <xacro:property name="shoulder_mass" value="0.37000" />
         <xacro:property name="upper_arm_mass" value="0.33930" />

File: melfa_description/urdf/rv80fr/rv80fr_macro.xacro (robot description, xacro)
@@ -12,5 +12,5 @@
     <xacro:macro name="rv80fr" params="parent prefix *origin">
         <!-- Inertial parameters -->
-        <xacro:property name="base_mass" value="0.4" />  <!-- These mass are INCORRRECT -->
+        <xacro:property name="base_mass" value="0.4" />  <!-- These mass are INCORRECT -->
         <xacro:property name="shoulder_mass" value="0.37000" />
         <xacro:property name="upper_arm_mass" value="0.33930" />

File: melfa_description/urdf/rv8crl/rv8crl_macro.xacro (robot description, xacro)
@@ -12,5 +12,5 @@
     <xacro:macro name="rv8crl" params="parent prefix *origin">
         <!-- Inertial parameters -->
-        <xacro:property name="base_mass" value="0.4" />  <!-- These mass are INCORRRECT -->
+        <xacro:property name="base_mass" value="0.4" />  <!-- These mass are INCORRECT -->
         <xacro:property name="shoulder_mass" value="0.37000" />
         <xacro:property name="upper_arm_mass" value="0.33930" />
